File: hardware/nuevipcbs/NuEVI.brd (EAGLE design)
At the start: 57.5 x 76.2 mm, 90 parts

Commit message: Added latest NuEVI schematic, board and gerber files.
Parts:
- added JP77, JP78: (no value), pinhead:1X01
- moved JP47 8.03 mm to (33.7, 8.26)
- moved JP68 2.54 mm to (43.8, 8.26)
- moved JP69 2.54 mm to (46.4, 8.26)
Connections:
- net GND: now also JP78.1
- net N$29: now also JP77.1
Routing:
- net N$22: track 61.5 -> 51.4 mm
- net N$29: track 50.1 -> 54.0 mm
- net N$42: track 40.9 -> 37.6 mm
Other:
- board text added: "BCV"
Changed lines of the file:
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@@
 <text x="10.16" y="19.685" size="1.016" layer="119" font="vector">47</text>
 <text x="10.16" y="17.145" size="1.016" layer="119" font="vector">47</text>
-<text x="40.64" y="3.175" size="1.016" layer="119" font="vector">A6</text>
+<text x="33.02" y="5.715" size="1.016" layer="119" font="vector">A6</text>
 <text x="1.905" y="26.035" size="1.016" layer="119" font="vector">A7</text>
 <text x="17.78" y="10.16" size="1.016" layer="119" font="vector">Vcc</text>
@@
 <wire x1="27.94" y1="71.12" x2="26.67" y2="69.85" width="0.254" layer="119"/>
 <text x="33.02" y="71.755" size="1.016" layer="119" font="vector">KEYS/ROLLERS</text>
-<text x="43.815" y="7.62" size="1.016" layer="119" font="vector">DAC</text>
-<text x="43.815" y="3.175" size="1.016" layer="119" font="vector">+</text>
-<text x="46.355" y="3.175" size="1.016" layer="119" font="vector">-</text>
+<text x="43.815" y="5.715" size="0.8128" layer="119" font="vector">DAC</text>
+<text x="42.545" y="5.715" size="1.016" layer="119" font="vector">+</text>
+<text x="46.355" y="5.715" size="1.016" layer="119" font="vector">-</text>
 <text x="15.24" y="50.8" size="1.016" layer="119" rot="R180">10K</text>
 <text x="15.24" y="40.64" size="1.016" layer="119" rot="R180">10K</text>
@@
 <text x="43.815" y="27.305" size="1.016" layer="119">SCL</text>
 <text x="34.925" y="27.305" size="1.016" layer="119">SDA</text>
+<text x="39.37" y="5.715" size="1.016" layer="119" font="vector">BCV</text>
+<text x="29.845" y="5.715" size="1.016" layer="119" font="vector">GND</text>
 </plain>
 <attributes>
@@
 <element name="U$1" library="Teensy_3_and_LC_Series_Boards_v1.4" package="TEENSY_3.0-3.2&amp;LC_DIL" value="TEENSY_LC_DIL" x="16.51" y="45.72"/>
 <element name="S1" library="switch" package="TL3XPO" value="TL36PO" x="3.81" y="55.245" rot="R90"/>
-<element name="JP47" library="pinhead" package="1X01" value="" x="41.275" y="5.715"/>
+<element name="JP47" library="pinhead" package="1X01" value="" x="33.655" y="8.255"/>
 <element name="JP48" library="pinhead" package="1X01" value="" x="2.54" y="28.575"/>
 <element name="JP49" library="pinhead" package="1X01" value="" x="20.32" y="8.255"/>
@@
 <element name="R4" library="resistor" package="0207/7" value="100" x="11.43" y="22.86"/>
 <element name="JP67" library="pinhead" package="1X01" value="" x="21.59" y="29.21"/>
-<element name="JP68" library="pinhead" package="1X01" value="" x="43.815" y="5.715"/>
-<element name="JP69" library="pinhead" package="1X01" value="" x="46.355" y="5.715"/>
+<element name="JP68" library="pinhead" package="1X01" value="" x="43.815" y="8.255"/>
+<element name="JP69" library="pinhead" package="1X01" value="" x="46.355" y="8.255"/>
 <element name="JP70" library="pinhead" package="1X01" value="" x="21.59" y="49.53"/>
 <element name="R5" library="resistor" package="0207/7" value="10K" x="16.51" y="40.64" rot="R270"/>
@@
 <element name="JP75" library="pinhead" package="1X01" value="" x="41.91" y="27.94"/>
 <element name="JP76" library="pinhead" package="1X01" value="" x="39.37" y="27.94"/>
+<element name="JP77" library="pinhead" package="1X01" value="" x="41.275" y="8.255"/>
+<element name="JP78" library="pinhead" package="1X01" value="" x="31.115" y="8.255"/>
 </elements>
 <signals>
@@
 <contactref element="U$1" pad="15/A1"/>
 <contactref element="JP27" pad="1"/>
-<wire x1="24.13" y1="34.29" x2="29.21" y2="29.21" width="0.4064" layer="16"/>
+<wire x1="24.13" y1="34.29" x2="29.21" y2="34.29" width="0.4064" layer="16"/>
 <wire x1="47.625" y1="70.485" x2="48.895" y2="71.755" width="0.4064" layer="16"/>
 <wire x1="48.895" y1="71.755" x2="52.705" y2="71.755" width="0.4064" layer="16"/>
 <wire x1="47.625" y1="70.485" x2="47.625" y2="29.21" width="0.4064" layer="16"/>
-<wire x1="29.21" y1="29.21" x2="33.02" y2="29.21" width="0.4064" layer="16"/>
-<wire x1="33.02" y1="29.21" x2="36.83" y2="25.4" width="0.4064" layer="16"/>
-<wire x1="36.83" y1="25.4" x2="43.815" y2="25.4" width="0.4064" layer="16"/>
+<wire x1="29.21" y1="34.29" x2="38.1" y2="25.4" width="0.4064" layer="16"/>
+<wire x1="38.1" y1="25.4" x2="43.815" y2="25.4" width="0.4064" layer="16"/>
 <wire x1="43.815" y1="25.4" x2="47.625" y2="29.21" width="0.4064" layer="16"/>
 </signal>
@@
 <contactref element="JP72" pad="1"/>
 <contactref element="JP74" pad="1"/>
+<contactref element="JP78" pad="1"/>
+<wire x1="15.24" y1="67.31" x2="17.78" y2="67.31" width="0" layer="19" extent="1-1"/>
+<wire x1="8.89" y1="62.23" x2="15.24" y2="67.31" width="0" layer="19" extent="1-1"/>
+<wire x1="5.08" y1="62.865" x2="8.89" y2="62.23" width="0" layer="19" extent="1-1"/>
+<wire x1="24.13" y1="59.69" x2="17.78" y2="67.31" width="0" layer="19" extent="1-1"/>
+<wire x1="5.08" y1="46.99" x2="8.89" y2="62.23" width="0" layer="19" extent="1-1"/>
+<wire x1="2.54" y1="33.655" x2="5.08" y2="46.99" width="0" layer="19" extent="1-1"/>
+<wire x1="16.51" y1="36.83" x2="2.54" y2="33.655" width="0" layer="19" extent="1-1"/>
+<wire x1="27.94" y1="39.37" x2="16.51" y2="36.83" width="0" layer="19" extent="1-1"/>
+<wire x1="36.957" y1="17.78" x2="27.94" y2="39.37" width="0" layer="19" extent="1-1"/>
+<wire x1="45.72" y1="16.51" x2="36.957" y2="17.78" width="0" layer="19" extent="1-1"/>
+<wire x1="45.72" y1="20.32" x2="45.72" y2="16.51" width="0" layer="19" extent="1-1"/>
+<wire x1="45.72" y1="12.7" x2="45.72" y2="16.51" width="0" layer="19" extent="1-1"/>
+<wire x1="46.355" y1="8.255" x2="45.72" y2="12.7" width="0" layer="19" extent="1-1"/>
+<wire x1="31.115" y1="8.255" x2="36.957" y2="17.78" width="0" layer="19" extent="1-1"/>
+<wire x1="20.32" y1="5.715" x2="31.115" y2="8.255" width="0" layer="19" extent="1-1"/>
+<wire x1="17.78" y1="5.715" x2="20.32" y2="5.715" width="0" layer="19" extent="1-1"/>
+<wire x1="15.24" y1="5.715" x2="17.78" y2="5.715" width="0" layer="19" extent="1-1"/>
+<wire x1="12.7" y1="5.715" x2="15.24" y2="5.715" width="0" layer="19" extent="1-1"/>
+<wire x1="7.62" y1="5.715" x2="12.7" y2="5.715" width="0" layer="19" extent="1-1"/>
+<wire x1="7.62" y1="8.255" x2="7.62" y2="5.715" width="0" layer="19" extent="1-1"/>
 </signal>
 <signal name="N$23">
@@
 <wire x1="33.02" y1="15.24" x2="34.29" y2="13.97" width="0.4064" layer="16"/>
 <wire x1="34.29" y1="13.97" x2="39.37" y2="13.97" width="0.4064" layer="16"/>
+<contactref element="JP77" pad="1"/>
+<wire x1="41.275" y1="8.255" x2="41.275" y2="9.525" width="0.4064" layer="1"/>
+<wire x1="41.275" y1="9.525" x2="39.37" y2="11.43" width="0.4064" layer="1"/>
 </signal>
 <signal name="N$12">
@@
 <wire x1="21.59" y1="25.4" x2="29.21" y2="25.4" width="0.4064" layer="16"/>
 <wire x1="29.21" y1="25.4" x2="30.48" y2="24.13" width="0.4064" layer="16"/>
-<wire x1="30.48" y1="24.13" x2="30.48" y2="8.89" width="0.4064" layer="16"/>
-<wire x1="41.275" y1="5.715" x2="33.655" y2="5.715" width="0.4064" layer="16"/>
-<wire x1="33.655" y1="5.715" x2="30.48" y2="8.89" width="0.4064" layer="16"/>
+<wire x1="30.48" y1="24.13" x2="30.48" y2="12.7" width="0.4064" layer="16"/>
+<wire x1="33.655" y1="9.525" x2="30.48" y2="12.7" width="0.4064" layer="16"/>
+<wire x1="33.655" y1="8.255" x2="33.655" y2="9.525" width="0.4064" layer="16"/>
 </signal>
 <signal name="N$31">
@@
 <contactref element="JP67" pad="1"/>
 <contactref element="JP68" pad="1"/>
-<wire x1="43.815" y1="5.715" x2="41.91" y2="7.62" width="0.4064" layer="16"/>
-<wire x1="41.91" y1="7.62" x2="34.29" y2="7.62" width="0.4064" layer="16"/>
-<wire x1="34.29" y1="7.62" x2="31.75" y2="10.16" width="0.4064" layer="16"/>
-<wire x1="31.75" y1="10.16" x2="31.75" y2="25.4" width="0.4064" layer="16"/>
+<wire x1="43.815" y1="8.255" x2="40.64" y2="11.43" width="0.4064" layer="16"/>
+<wire x1="40.64" y1="11.43" x2="34.29" y2="11.43" width="0.4064" layer="16"/>
+<wire x1="34.29" y1="11.43" x2="31.75" y2="13.97" width="0.4064" layer="16"/>
+<wire x1="31.75" y1="13.97" x2="31.75" y2="25.4" width="0.4064" layer="16"/>
 <wire x1="31.75" y1="25.4" x2="30.48" y2="26.67" width="0.4064" layer="16"/>
 <wire x1="30.48" y1="26.67" x2="24.13" y2="26.67" width="0.4064" layer="16"/>
