File: hardware/nuevipcbs/NuEVI.sch (EAGLE design)
At the start: 90 parts

Commit message: Added latest NuEVI schematic, board and gerber files.
Parts:
- added JP77, JP78: (no value), pinhead:PINHD-1X1
Connections:
- net GND: now also JP78.1
- net N$29: now also JP77.1
Changed lines of the file:
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@@
 <part name="JP75" library="pinhead" deviceset="PINHD-1X1" device=""/>
 <part name="JP76" library="pinhead" deviceset="PINHD-1X1" device=""/>
+<part name="JP77" library="pinhead" deviceset="PINHD-1X1" device=""/>
+<part name="JP78" library="pinhead" deviceset="PINHD-1X1" device=""/>
 </parts>
 <sheets>
@@
 <instance part="JP75" gate="G$1" x="63.5" y="60.96"/>
 <instance part="JP76" gate="G$1" x="63.5" y="38.1"/>
+<instance part="JP77" gate="G$1" x="76.454" y="-35.56"/>
+<instance part="JP78" gate="G$1" x="76.454" y="-50.8"/>
 </instances>
 <busses>
@@
 <pinref part="PS1" gate="G$1" pin="GND"/>
 <wire x1="53.34" y1="-50.8" x2="40.64" y2="-50.8" width="0.1524" layer="91"/>
-<wire x1="40.64" y1="-50.8" x2="40.64" y2="-40.64" width="0.1524" layer="91"/>
 <pinref part="C1" gate="G$1" pin="1"/>
 <junction x="68.58" y="-5.08"/>
@@
 <wire x1="78.74" y1="-5.08" x2="88.9" y2="-5.08" width="0.1524" layer="91"/>
 <wire x1="106.68" y1="-5.08" x2="106.68" y2="-30.48" width="0.1524" layer="91"/>
+<wire x1="73.914" y1="-50.8" x2="53.34" y2="-50.8" width="0.1524" layer="91"/>
+<wire x1="40.64" y1="-50.8" x2="40.64" y2="-40.64" width="0.1524" layer="91"/>
+<pinref part="JP78" gate="G$1" pin="1"/>
 </segment>
 <segment>
@@
 <pinref part="C3" gate="G$1" pin="2"/>
 <junction x="83.82" y="-25.4"/>
-</segment>
-</net>
+<wire x1="66.04" y1="-35.56" x2="66.04" y2="-25.4" width="0.1524" layer="91"/>
+<pinref part="JP77" gate="G$1" pin="1"/>
+<wire x1="66.04" y1="-35.56" x2="73.914" y2="-35.56" width="0.1524" layer="91"/>
+</segment>
+</net>
